Commit message: feat(tianyi2): render calibrated hand and lift skeleton

File: x-humanoid/tianyi2.0/resource/tianyi2_model.urdf (robot description, URDF)
Before this commit: robot Tianyi2Pro, 24 links, 23 joints
Links:
- removed link chassis_link
- removed link left_hip_pitch_link
- removed link left_knee_pitch_link
- added link base_center_link, mass 15.0
- added link base_heading_apex_link, mass 0.02
- added link base_heading_close_link, mass 0.02
- added link base_heading_tail_link, mass 0.02
- added link base_left_link, mass 0.1
- added link base_rear_link, mass 0.1
- added link head_tip_link, mass 0.2
- added link hip_pitch_link, mass 2.0
- added link knee_base_link, mass 1.5
- added link left_hand_index_distal_link, mass 0.02
- added link left_hand_index_link, mass 0.02
- added link left_hand_index_tip_link, mass 0.01
- added link left_hand_little_distal_link, mass 0.02
- added link left_hand_little_link, mass 0.02
- added link left_hand_little_tip_link, mass 0.01
- added link left_hand_middle_distal_link, mass 0.02
- added link left_hand_middle_link, mass 0.02
- added link left_hand_middle_tip_link, mass 0.01
- added link left_hand_ring_distal_link, mass 0.02
- added link left_hand_ring_link, mass 0.02
- added link left_hand_ring_tip_link, mass 0.01
- added link left_hand_thumb_bend_link, mass 0.02
- added link left_hand_thumb_rotation_link, mass 0.02
- added link left_hand_thumb_tip_link, mass 0.01
- added link left_palm_link, mass 0.15
- added link right_hand_index_distal_link, mass 0.02
- added link right_hand_index_link, mass 0.02
- added link right_hand_index_tip_link, mass 0.01
- added link right_hand_little_distal_link, mass 0.02
- added link right_hand_little_link, mass 0.02
- added link right_hand_little_tip_link, mass 0.01
- added link right_hand_middle_distal_link, mass 0.02
- added link right_hand_middle_link, mass 0.02
- added link right_hand_middle_tip_link, mass 0.01
- added link right_hand_ring_distal_link, mass 0.02
- added link right_hand_ring_link, mass 0.02
- added link right_hand_ring_tip_link, mass 0.01
- added link right_hand_thumb_bend_link, mass 0.02
- added link right_hand_thumb_rotation_link, mass 0.02
- added link right_hand_thumb_tip_link, mass 0.01
- added link right_palm_link, mass 0.15
Joints:
- removed joint chassis_to_pelvis
- removed joint left_hip_pitch_joint
- removed joint left_knee_pitch_joint
- added joint base_center_to_left: type fixed, parent base_center_link, child base_left_link, origin xyz=0 0.24 0 rpy=0 0 0
- added joint base_center_to_rear: type fixed, parent base_center_link, child base_rear_link, origin xyz=-0.32 0 0 rpy=0 0 0
- added joint base_heading_apex_to_tail: type fixed, parent base_heading_apex_link, child base_heading_tail_link, origin xyz=-0.30 -0.24 0 rpy=0 0 0
- added joint base_heading_tail_to_close: type fixed, parent base_heading_tail_link, child base_heading_close_link, origin xyz=0 0.48 -0.03 rpy=0 0 0
- added joint base_left_to_heading_apex: type fixed, parent base_left_link, child base_heading_apex_link, origin xyz=0.30 -0.24 0.03 rpy=0 0 0
- added joint head_to_tip: type fixed, parent head_roll_link, child head_tip_link, origin xyz=0 0 0.12 rpy=0 0 0
- added joint hip_pitch_joint: type revolute, parent knee_base_link, child hip_pitch_link, origin xyz=-0.225 0 0.390 rpy=0 0 0, axis 0 1 0, limit lower=-0.227 upper=3.142 effort=332 velocity=3.93
- added joint hip_to_waist: type fixed, parent hip_pitch_link, child pelvis_link, origin xyz=0.225 0 0.390 rpy=0 0 0
- added joint knee_pitch_joint: type revolute, parent base_center_link, child knee_base_link, origin xyz=0 0 0.36 rpy=0 0 0, axis 0 1 0, limit lower=-1.571 upper=2.793 effort=332 velocity=3.93
- added joint left_hand_index_distal_joint: type revolute, parent left_hand_index_link, child left_hand_index_distal_link, origin xyz=0 0 -0.070 rpy=0 0 0, axis 0 1 0, limit lower=-1.571 upper=0 effort=2 velocity=4
- added joint left_hand_index_joint: type revolute, parent left_palm_link, child left_hand_index_link, origin xyz=0 0.015 -0.025 rpy=0 0 0, axis 0 1 0, limit lower=-1.571 upper=0 effort=2 velocity=4
- added joint left_hand_index_tip: type fixed, parent left_hand_index_distal_link, child left_hand_index_tip_link, origin xyz=0 0 -0.070 rpy=0 0 0
- added joint left_hand_little_distal_joint: type revolute, parent left_hand_little_link, child left_hand_little_distal_link, origin xyz=0 0 -0.060 rpy=0 0 0, axis 0 1 0, limit lower=-1.571 upper=0 effort=2 velocity=4
- added joint left_hand_little_joint: type revolute, parent left_palm_link, child left_hand_little_link, origin xyz=0 -0.03 -0.02 rpy=0 0 0, axis 0 1 0, limit lower=-1.571 upper=0 effort=2 velocity=4
- added joint left_hand_little_tip: type fixed, parent left_hand_little_distal_link, child left_hand_little_tip_link, origin xyz=0 0 -0.060 rpy=0 0 0
- added joint left_hand_middle_distal_joint: type revolute, parent left_hand_middle_link, child left_hand_middle_distal_link, origin xyz=0 0 -0.075 rpy=0 0 0, axis 0 1 0, limit lower=-1.571 upper=0 effort=2 velocity=4
- added joint left_hand_middle_joint: type revolute, parent left_palm_link, child left_hand_middle_link, origin xyz=0 0 -0.028 rpy=0 0 0, axis 0 1 0, limit lower=-1.571 upper=0 effort=2 velocity=4
- added joint left_hand_middle_tip: type fixed, parent left_hand_middle_distal_link, child left_hand_middle_tip_link, origin xyz=0 0 -0.075 rpy=0 0 0
- added joint left_hand_ring_distal_joint: type revolute, parent left_hand_ring_link, child left_hand_ring_distal_link, origin xyz=0 0 -0.070 rpy=0 0 0, axis 0 1 0, limit lower=-1.571 upper=0 effort=2 velocity=4
- added joint left_hand_ring_joint: type revolute, parent left_palm_link, child left_hand_ring_link, origin xyz=0 -0.015 -0.025 rpy=0 0 0, axis 0 1 0, limit lower=-1.571 upper=0 effort=2 velocity=4
- added joint left_hand_ring_tip: type fixed, parent left_hand_ring_distal_link, child left_hand_ring_tip_link, origin xyz=0 0 -0.070 rpy=0 0 0
- added joint left_hand_thumb_bend_joint: type revolute, parent left_hand_thumb_rotation_link, child left_hand_thumb_bend_link, origin xyz=0 0.025 -0.02 rpy=0 0 0, axis -1 0 0, limit lower=0 upper=1.571 effort=2 velocity=4
- added joint left_hand_thumb_rotation_joint: type revolute, parent left_palm_link, child left_hand_thumb_rotation_link, origin xyz=0 0.035 -0.015 rpy=0 0 0, axis 0 0 -1, limit lower=0 upper=1.571 effort=2 velocity=4
- added joint left_hand_thumb_tip: type fixed, parent left_hand_thumb_bend_link, child left_hand_thumb_tip_link, origin xyz=0.006 0.035 -0.020 rpy=0 0 0
- added joint left_wrist_to_palm: type fixed, parent left_wrist_roll_link, child left_palm_link, origin xyz=0 0 0 rpy=0 0 -1.570796
- added joint right_hand_index_distal_joint: type revolute, parent right_hand_index_link, child right_hand_index_distal_link, origin xyz=0 0 -0.070 rpy=0 0 0, axis 0 1 0, limit lower=-1.571 upper=0 effort=2 velocity=4
- added joint right_hand_index_joint: type revolute, parent right_palm_link, child right_hand_index_link, origin xyz=0 0.015 -0.025 rpy=0 0 0, axis 0 1 0, limit lower=-1.571 upper=0 effort=2 velocity=4
- added joint right_hand_index_tip: type fixed, parent right_hand_index_distal_link, child right_hand_index_tip_link, origin xyz=0 0 -0.070 rpy=0 0 0
- added joint right_hand_little_distal_joint: type revolute, parent right_hand_little_link, child right_hand_little_distal_link, origin xyz=0 0 -0.060 rpy=0 0 0, axis 0 1 0, limit lower=-1.571 upper=0 effort=2 velocity=4
- added joint right_hand_little_joint: type revolute, parent right_palm_link, child right_hand_little_link, origin xyz=0 -0.03 -0.02 rpy=0 0 0, axis 0 1 0, limit lower=-1.571 upper=0 effort=2 velocity=4
- added joint right_hand_little_tip: type fixed, parent right_hand_little_distal_link, child right_hand_little_tip_link, origin xyz=0 0 -0.060 rpy=0 0 0
- added joint right_hand_middle_distal_joint: type revolute, parent right_hand_middle_link, child right_hand_middle_distal_link, origin xyz=0 0 -0.075 rpy=0 0 0, axis 0 1 0, limit lower=-1.571 upper=0 effort=2 velocity=4
- added joint right_hand_middle_joint: type revolute, parent right_palm_link, child right_hand_middle_link, origin xyz=0 0 -0.028 rpy=0 0 0, axis 0 1 0, limit lower=-1.571 upper=0 effort=2 velocity=4
- added joint right_hand_middle_tip: type fixed, parent right_hand_middle_distal_link, child right_hand_middle_tip_link, origin xyz=0 0 -0.075 rpy=0 0 0
- added joint right_hand_ring_distal_joint: type revolute, parent right_hand_ring_link, child right_hand_ring_distal_link, origin xyz=0 0 -0.070 rpy=0 0 0, axis 0 1 0, limit lower=-1.571 upper=0 effort=2 velocity=4
- added joint right_hand_ring_joint: type revolute, parent right_palm_link, child right_hand_ring_link, origin xyz=0 -0.015 -0.025 rpy=0 0 0, axis 0 1 0, limit lower=-1.571 upper=0 effort=2 velocity=4
- added joint right_hand_ring_tip: type fixed, parent right_hand_ring_distal_link, child right_hand_ring_tip_link, origin xyz=0 0 -0.070 rpy=0 0 0
- added joint right_hand_thumb_bend_joint: type revolute, parent right_hand_thumb_rotation_link, child right_hand_thumb_bend_link, origin xyz=0 -0.025 -0.02 rpy=0 0 0, axis 1 0 0, limit lower=0 upper=1.571 effort=2 velocity=4
- added joint right_hand_thumb_rotation_joint: type revolute, parent right_palm_link, child right_hand_thumb_rotation_link, origin xyz=0 -0.035 -0.015 rpy=0 0 0, axis 0 0 1, limit lower=0 upper=1.571 effort=2 velocity=4
- added joint right_hand_thumb_tip: type fixed, parent right_hand_thumb_bend_link, child right_hand_thumb_tip_link, origin xyz=0.006 -0.035 -0.020 rpy=0 0 0
- added joint right_wrist_to_palm: type fixed, parent right_wrist_roll_link, child right_palm_link, origin xyz=0 0 0 rpy=0 0 1.570796
- joint head_pitch_joint: origin xyz=0 0 0.05 rpy=0 0 0 -> xyz=0 0 0 rpy=0 0 0
- joint head_roll_joint: origin xyz=0 0 0.05 rpy=0 0 0 -> xyz=0 0 0 rpy=0 0 0
- joint left_elbow_pitch_joint: origin xyz=0 0 -0.22 rpy=0 0 0 -> xyz=0 0 -0.30 rpy=0 0 0
- joint left_shoulder_pitch_joint: origin xyz=0 0.18 0.05 rpy=0 0 0 -> xyz=0 0.22 -0.02 rpy=0 0 0
- joint left_shoulder_roll_joint: origin xyz=0 0.05 0 rpy=0 0 0 -> xyz=0 0 0 rpy=0 0 0
- joint left_shoulder_yaw_joint: origin xyz=0 0.05 0 rpy=0 0 0 -> xyz=0 0 0 rpy=0 0 0
- joint left_wrist_pitch_joint: origin xyz=0 0 -0.05 rpy=0 0 0 -> xyz=0 0 0 rpy=0 0 0
- joint left_wrist_roll_joint: origin xyz=0 0 -0.05 rpy=0 0 0 -> xyz=0 0 0 rpy=0 0 0
- joint left_wrist_yaw_joint: origin xyz=0 0 -0.2 rpy=0 0 0 -> xyz=0 0 -0.24 rpy=0 0 0
- joint right_elbow_pitch_joint: origin xyz=0 0 -0.22 rpy=0 0 0 -> xyz=0 0 -0.30 rpy=0 0 0
- joint right_shoulder_pitch_joint: origin xyz=0 -0.18 0.05 rpy=0 0 0 -> xyz=0 -0.22 -0.02 rpy=0 0 0
- joint right_shoulder_roll_joint: origin xyz=0 -0.05 0 rpy=0 0 0 -> xyz=0 0 0 rpy=0 0 0
- joint right_shoulder_yaw_joint: origin xyz=0 -0.05 0 rpy=0 0 0 -> xyz=0 0 0 rpy=0 0 0
- joint right_wrist_pitch_joint: origin xyz=0 0 -0.05 rpy=0 0 0 -> xyz=0 0 0 rpy=0 0 0
- joint right_wrist_roll_joint: origin xyz=0 0 -0.05 rpy=0 0 0 -> xyz=0 0 0 rpy=0 0 0
- joint right_wrist_yaw_joint: origin xyz=0 0 -0.2 rpy=0 0 0 -> xyz=0 0 -0.24 rpy=0 0 0
- joint waist_pitch_joint: limit lower=-0.785 upper=2.094 effort=332 velocity=3.93 -> lower=-1.745 upper=2.094 effort=332 velocity=3.93; origin xyz=0 0 0.05 rpy=0 0 0 -> xyz=0 0 0 rpy=0 0 0
- joint waist_to_torso: origin xyz=0 0 0.3 rpy=0 0 0 -> xyz=0 0 0.36 rpy=0 0 0
- joint waist_yaw_joint: origin xyz=0 0 0.1 rpy=0 0 0 -> xyz=0 0 0 rpy=0 0 0

Commit message: fix(tianyi2): reduce joints latency and correct palm length

File: x-humanoid/tianyi2.0/resource/tianyi2_model.urdf (robot description, URDF)
Before this commit: robot Tianyi2Pro, 62 links, 61 joints
Joints:
- joint left_hand_index_distal_joint: origin xyz=0 0 -0.070 rpy=0 0 0 -> xyz=0 0 -0.035 rpy=0 0 0
- joint left_hand_index_joint: origin xyz=0 0.015 -0.025 rpy=0 0 0 -> xyz=0 0.015 -0.060 rpy=0 0 0
- joint left_hand_little_distal_joint: origin xyz=0 0 -0.060 rpy=0 0 0 -> xyz=0 0 -0.030 rpy=0 0 0
- joint left_hand_little_joint: origin xyz=0 -0.03 -0.02 rpy=0 0 0 -> xyz=0 -0.03 -0.050 rpy=0 0 0
- joint left_hand_middle_distal_joint: origin xyz=0 0 -0.075 rpy=0 0 0 -> xyz=0 0 -0.0375 rpy=0 0 0
- joint left_hand_middle_joint: origin xyz=0 0 -0.028 rpy=0 0 0 -> xyz=0 0 -0.0655 rpy=0 0 0
- joint left_hand_ring_distal_joint: origin xyz=0 0 -0.070 rpy=0 0 0 -> xyz=0 0 -0.035 rpy=0 0 0
- joint left_hand_ring_joint: origin xyz=0 -0.015 -0.025 rpy=0 0 0 -> xyz=0 -0.015 -0.060 rpy=0 0 0
- joint right_hand_index_distal_joint: origin xyz=0 0 -0.070 rpy=0 0 0 -> xyz=0 0 -0.035 rpy=0 0 0
- joint right_hand_index_joint: origin xyz=0 0.015 -0.025 rpy=0 0 0 -> xyz=0 0.015 -0.060 rpy=0 0 0
- joint right_hand_little_distal_joint: origin xyz=0 0 -0.060 rpy=0 0 0 -> xyz=0 0 -0.030 rpy=0 0 0
- joint right_hand_little_joint: origin xyz=0 -0.03 -0.02 rpy=0 0 0 -> xyz=0 -0.03 -0.050 rpy=0 0 0
- joint right_hand_middle_distal_joint: origin xyz=0 0 -0.075 rpy=0 0 0 -> xyz=0 0 -0.0375 rpy=0 0 0
- joint right_hand_middle_joint: origin xyz=0 0 -0.028 rpy=0 0 0 -> xyz=0 0 -0.0655 rpy=0 0 0
- joint right_hand_ring_distal_joint: origin xyz=0 0 -0.070 rpy=0 0 0 -> xyz=0 0 -0.035 rpy=0 0 0
- joint right_hand_ring_joint: origin xyz=0 -0.015 -0.025 rpy=0 0 0 -> xyz=0 -0.015 -0.060 rpy=0 0 0

Commit message: fix(tianyi2): mirror right-hand finger placement

File: x-humanoid/tianyi2.0/resource/tianyi2_model.urdf (robot description, URDF)
Before this commit: robot Tianyi2Pro, 62 links, 61 joints
Joints:
- joint right_hand_index_joint: origin xyz=0 0.015 -0.060 rpy=0 0 0 -> xyz=0 -0.015 -0.060 rpy=0 0 0
- joint right_hand_little_joint: origin xyz=0 -0.03 -0.050 rpy=0 0 0 -> xyz=0 0.030 -0.050 rpy=0 0 0
- joint right_hand_ring_joint: origin xyz=0 -0.015 -0.060 rpy=0 0 0 -> xyz=0 0.015 -0.060 rpy=0 0 0

Commit message: fix(tianyi2): shorten four-finger distal segments

File: x-humanoid/tianyi2.0/resource/tianyi2_model.urdf (robot description, URDF)
Before this commit: robot Tianyi2Pro, 62 links, 61 joints
Joints:
- joint left_hand_index_tip: origin xyz=0 0 -0.070 rpy=0 0 0 -> xyz=0 0 -0.035 rpy=0 0 0
- joint left_hand_little_tip: origin xyz=0 0 -0.060 rpy=0 0 0 -> xyz=0 0 -0.030 rpy=0 0 0
- joint left_hand_middle_tip: origin xyz=0 0 -0.075 rpy=0 0 0 -> xyz=0 0 -0.0375 rpy=0 0 0
- joint left_hand_ring_tip: origin xyz=0 0 -0.070 rpy=0 0 0 -> xyz=0 0 -0.035 rpy=0 0 0
- joint right_hand_index_tip: origin xyz=0 0 -0.070 rpy=0 0 0 -> xyz=0 0 -0.035 rpy=0 0 0
- joint right_hand_little_tip: origin xyz=0 0 -0.060 rpy=0 0 0 -> xyz=0 0 -0.030 rpy=0 0 0
- joint right_hand_middle_tip: origin xyz=0 0 -0.075 rpy=0 0 0 -> xyz=0 0 -0.0375 rpy=0 0 0
- joint right_hand_ring_tip: origin xyz=0 0 -0.070 rpy=0 0 0 -> xyz=0 0 -0.035 rpy=0 0 0

Commit message: fix(tianyi2): set inward thumb rest rotation

File: x-humanoid/tianyi2.0/resource/tianyi2_model.urdf (robot description, URDF)
Before this commit: robot Tianyi2Pro, 62 links, 61 joints
Joints:
- joint left_hand_thumb_rotation_joint: origin xyz=0 0.035 -0.015 rpy=0 0 0 -> xyz=0 0.035 -0.015 rpy=0 0 -0.349066
- joint right_hand_thumb_rotation_joint: origin xyz=0 -0.035 -0.015 rpy=0 0 0 -> xyz=0 -0.035 -0.015 rpy=0 0 0.349066
