Commit message: fix(unitree): harden AS2W deployment and model resources

File: unitree/as2w/resource/as2w.urdf (robot description, URDF)
Before this commit: robot AS2W, 18 links, 17 joints
Links:
- link FL_calf: geometry 
- link FL_foot: geometry 
- link FL_hip: geometry 
- link FL_thigh: geometry 
- link FR_calf: geometry 
- link FR_foot: geometry 
- link FR_hip: geometry 
- link FR_thigh: geometry 
- link JT128: geometry 
- link RL_calf: geometry 
- link RL_foot: geometry 
- link RL_hip: geometry 
- link RL_thigh: geometry 
- link RR_calf: geometry 
- link RR_foot: geometry 
- link RR_hip: geometry 
- link RR_thigh: geometry 
- link base_link: geometry 

Commit message: fix(as2w): add renderable robot geometry

File: unitree/as2w/resource/as2w.urdf (robot description, URDF)
Before this commit: robot AS2W, 18 links, 17 joints
Links:
- link FL_calf: geometry visual box size=0.09 0.09 0.24
- link FL_foot: geometry visual cylinder length=0.12 radius=0.055
- link FL_hip: geometry visual cylinder length=0.10 radius=0.055
- link FL_thigh: geometry visual box size=0.10 0.20 0.25
- link FR_calf: geometry visual box size=0.09 0.09 0.24
- link FR_foot: geometry visual cylinder length=0.12 radius=0.055
- link FR_hip: geometry visual cylinder length=0.10 radius=0.055
- link FR_thigh: geometry visual box size=0.10 0.20 0.25
- link JT128: geometry visual box size=0.16 0.12 0.10
- link RL_calf: geometry visual box size=0.09 0.09 0.24
- link RL_foot: geometry visual cylinder length=0.12 radius=0.055
- link RL_hip: geometry visual cylinder length=0.10 radius=0.055
- link RL_thigh: geometry visual box size=0.10 0.20 0.25
- link RR_calf: geometry visual box size=0.09 0.09 0.24
- link RR_foot: geometry visual cylinder length=0.12 radius=0.055
- link RR_hip: geometry visual cylinder length=0.10 radius=0.055
- link RR_thigh: geometry visual box size=0.10 0.20 0.25
- link base_link: geometry visual box size=0.42 0.28 0.12

Commit message: fix(as2w): expose wheel joints to legacy skeleton clients

File: unitree/as2w/resource/as2w.urdf (robot description, URDF)
Before this commit: robot AS2W, 18 links, 17 joints
Joints:
- joint FL_foot: limit effort=15 velocity=98.47 -> lower=-1000000 upper=1000000 effort=15 velocity=98.47; type continuous -> revolute
- joint FR_foot: limit effort=15 velocity=98.47 -> lower=-1000000 upper=1000000 effort=15 velocity=98.47; type continuous -> revolute
- joint RL_foot: limit effort=15 velocity=98.47 -> lower=-1000000 upper=1000000 effort=15 velocity=98.47; type continuous -> revolute
- joint RR_foot: limit effort=15 velocity=98.47 -> lower=-1000000 upper=1000000 effort=15 velocity=98.47; type continuous -> revolute

Commit message: fix(as2w): restore official continuous wheel joints

File: unitree/as2w/resource/as2w.urdf (robot description, URDF)
Before this commit: robot AS2W, 18 links, 17 joints
Joints:
- joint FL_foot: limit lower=-1000000 upper=1000000 effort=15 velocity=98.47 -> effort=15 velocity=98.47; type revolute -> continuous
- joint FR_foot: limit lower=-1000000 upper=1000000 effort=15 velocity=98.47 -> effort=15 velocity=98.47; type revolute -> continuous
- joint RL_foot: limit lower=-1000000 upper=1000000 effort=15 velocity=98.47 -> effort=15 velocity=98.47; type revolute -> continuous
- joint RR_foot: limit lower=-1000000 upper=1000000 effort=15 velocity=98.47 -> effort=15 velocity=98.47; type revolute -> continuous
