Commit message: feat(tron2): show gripper outlines and simplify arm actions

File: limx/tron2/resource/tron2_dach.urdf (robot description, URDF)
Before this commit: robot robot_description/tron2/DACH_TRON2A, 25 links, 24 joints
Links:
- added link display_hand_gripper_L_a_base_Link
- added link display_hand_gripper_L_a_tip_Link
- added link display_hand_gripper_L_b_base_Link
- added link display_hand_gripper_L_b_tip_Link
- added link display_hand_gripper_R_a_base_Link
- added link display_hand_gripper_R_a_tip_Link
- added link display_hand_gripper_R_b_base_Link
- added link display_hand_gripper_R_b_tip_Link
Joints:
- added joint display_hand_gripper_L_a_base_Joint: type fixed, parent grasper_L_Link, child display_hand_gripper_L_a_base_Link, origin xyz=0 0.025 0 rpy=0 0 0
- added joint display_hand_gripper_L_a_tip_Joint: type fixed, parent display_hand_gripper_L_a_base_Link, child display_hand_gripper_L_a_tip_Link, origin xyz=0 0 -0.065 rpy=0 0 0
- added joint display_hand_gripper_L_b_base_Joint: type fixed, parent grasper_L_Link, child display_hand_gripper_L_b_base_Link, origin xyz=0 -0.025 0 rpy=0 0 0
- added joint display_hand_gripper_L_b_tip_Joint: type fixed, parent display_hand_gripper_L_b_base_Link, child display_hand_gripper_L_b_tip_Link, origin xyz=0 0 -0.065 rpy=0 0 0
- added joint display_hand_gripper_R_a_base_Joint: type fixed, parent grasper_R_Link, child display_hand_gripper_R_a_base_Link, origin xyz=0 0.025 0 rpy=0 0 0
- added joint display_hand_gripper_R_a_tip_Joint: type fixed, parent display_hand_gripper_R_a_base_Link, child display_hand_gripper_R_a_tip_Link, origin xyz=0 0 -0.065 rpy=0 0 0
- added joint display_hand_gripper_R_b_base_Joint: type fixed, parent grasper_R_Link, child display_hand_gripper_R_b_base_Link, origin xyz=0 -0.025 0 rpy=0 0 0
- added joint display_hand_gripper_R_b_tip_Joint: type fixed, parent display_hand_gripper_R_b_base_Link, child display_hand_gripper_R_b_tip_Link, origin xyz=0 0 -0.065 rpy=0 0 0

Commit message: fix(tron2): show stock grippers closed by default

File: limx/tron2/resource/tron2_dach.urdf (robot description, URDF)
Before this commit: robot robot_description/tron2/DACH_TRON2A, 33 links, 32 joints
Joints:
- joint display_hand_gripper_L_a_base_Joint: origin xyz=0 0.025 0 rpy=0 0 0 -> xyz=0 0.004 0 rpy=0 0 0
- joint display_hand_gripper_L_b_base_Joint: origin xyz=0 -0.025 0 rpy=0 0 0 -> xyz=0 -0.004 0 rpy=0 0 0
- joint display_hand_gripper_R_a_base_Joint: origin xyz=0 0.025 0 rpy=0 0 0 -> xyz=0 0.004 0 rpy=0 0 0
- joint display_hand_gripper_R_b_base_Joint: origin xyz=0 -0.025 0 rpy=0 0 0 -> xyz=0 -0.004 0 rpy=0 0 0
