Commit message: fix A3 pose audio and O10 hand mapping

File: agibot/A3/resource/a3_ultra.urdf (robot description, URDF)
Before this commit: robot a3_ultra, 47 links, 46 joints
Links:
- added link left_hand_channel_5
- added link left_hand_channel_6
- added link left_hand_channel_7
- added link left_hand_channel_8
- added link left_hand_channel_9
- added link right_hand_channel_5
- added link right_hand_channel_6
- added link right_hand_channel_7
- added link right_hand_channel_8
- added link right_hand_channel_9
Joints:
- removed joint left_hand_joint_0
- removed joint left_hand_joint_1
- removed joint left_hand_joint_2
- removed joint left_hand_joint_3
- removed joint left_hand_joint_4
- removed joint right_hand_joint_0
- removed joint right_hand_joint_1
- removed joint right_hand_joint_2
- removed joint right_hand_joint_3
- removed joint right_hand_joint_4
- added joint left_index_bent_1: type revolute, parent left_hand_channel_3, child left_hand_channel_4, axis 0 0 1, limit lower=0 upper=4096 effort=0 velocity=0
- added joint left_index_wiggles_0: type revolute, parent left_hand_link, child left_hand_channel_3, axis 0 1 0, limit lower=0 upper=4096 effort=0 velocity=0
- added joint left_middle_bent: type revolute, parent left_hand_link, child left_hand_channel_5, axis 0 0 1, limit lower=0 upper=4096 effort=0 velocity=0
- added joint left_pinky_bent_1: type revolute, parent left_hand_channel_8, child left_hand_channel_9, axis 0 0 1, limit lower=0 upper=4096 effort=0 velocity=0
- added joint left_pinky_wiggles_0: type revolute, parent left_hand_link, child left_hand_channel_8, axis 0 1 0, limit lower=0 upper=4096 effort=0 velocity=0
- added joint left_ring_bent_1: type revolute, parent left_hand_channel_6, child left_hand_channel_7, axis 0 0 1, limit lower=0 upper=4096 effort=0 velocity=0
- added joint left_ring_wiggles_0: type revolute, parent left_hand_link, child left_hand_channel_6, axis 0 1 0, limit lower=0 upper=4096 effort=0 velocity=0
- added joint left_thumb_bent_2: type revolute, parent left_hand_channel_1, child left_hand_channel_2, axis 0 0 1, limit lower=0 upper=4096 effort=0 velocity=0
- added joint left_thumb_roration_0: type revolute, parent left_hand_link, child left_hand_channel_0, axis 1 0 0, limit lower=0 upper=4096 effort=0 velocity=0
- added joint left_thumb_wiggles_1: type revolute, parent left_hand_channel_0, child left_hand_channel_1, axis 0 1 0, limit lower=0 upper=4096 effort=0 velocity=0
- added joint right_index_bent_1: type revolute, parent right_hand_channel_3, child right_hand_channel_4, axis 0 0 1, limit lower=0 upper=4096 effort=0 velocity=0
- added joint right_index_wiggles_0: type revolute, parent right_hand_link, child right_hand_channel_3, axis 0 1 0, limit lower=0 upper=4096 effort=0 velocity=0
- added joint right_middle_bent: type revolute, parent right_hand_link, child right_hand_channel_5, axis 0 0 1, limit lower=0 upper=4096 effort=0 velocity=0
- added joint right_pinky_bent_1: type revolute, parent right_hand_channel_8, child right_hand_channel_9, axis 0 0 1, limit lower=0 upper=4096 effort=0 velocity=0
- added joint right_pinky_wiggles_0: type revolute, parent right_hand_link, child right_hand_channel_8, axis 0 1 0, limit lower=0 upper=4096 effort=0 velocity=0
- added joint right_ring_bent_1: type revolute, parent right_hand_channel_6, child right_hand_channel_7, axis 0 0 1, limit lower=0 upper=4096 effort=0 velocity=0
- added joint right_ring_wiggles_0: type revolute, parent right_hand_link, child right_hand_channel_6, axis 0 1 0, limit lower=0 upper=4096 effort=0 velocity=0
- added joint right_thumb_bent_2: type revolute, parent right_hand_channel_1, child right_hand_channel_2, axis 0 0 1, limit lower=0 upper=4096 effort=0 velocity=0
- added joint right_thumb_rotation_0: type revolute, parent right_hand_link, child right_hand_channel_0, axis 1 0 0, limit lower=0 upper=4096 effort=0 velocity=0
- added joint right_thumb_wiggles_1: type revolute, parent right_hand_channel_0, child right_hand_channel_1, axis 0 1 0, limit lower=0 upper=4096 effort=0 velocity=0
