Commit message: Improve A3 camera relay and robot model

File: agibot/A3/resource/a3_ultra.urdf (robot description, URDF)
Before this commit: robot a3_ultra, 57 links, 56 joints
Links:
- removed link head_pitch_link
- removed link head_yaw_link
- removed link imu_in_pelvis_link
- removed link imu_in_torso_link
- removed link left_ankle_pitch_link
- removed link left_elbow_link
- removed link left_foot
- removed link left_hand_link
- removed link left_hip_pitch_link
- removed link left_hip_roll_link
- removed link left_hip_yaw_link
- removed link left_knee_link
- removed link left_shoulder_pitch_link
- removed link left_shoulder_roll_link
- removed link left_shoulder_yaw_link
- removed link left_wrist_pitch_link
- removed link left_wrist_roll_link
- removed link left_wrist_yaw_link
- removed link pelvis
- removed link right_ankle_pitch_link
- removed link right_elbow_link
- removed link right_foot
- removed link right_hand_link
- removed link right_hip_pitch_link
- removed link right_hip_roll_link
- removed link right_hip_yaw_link
- removed link right_knee_link
- removed link right_shoulder_pitch_link
- removed link right_shoulder_roll_link
- removed link right_shoulder_yaw_link
- removed link right_wrist_pitch_link
- removed link right_wrist_roll_link
- removed link right_wrist_yaw_link
- removed link torso
- removed link waist_pitch_link
- removed link waist_roll_link
- removed link waist_yaw_link
- added link D415_in_torso_Link, mass 0; collision mesh filename=../meshes/D415_in_torso_Link.STL; visual mesh filename=../meshes/D415_in_torso_Link.STL
- added link D457_in_torso_Link, mass 0; collision mesh filename=../meshes/D457_in_torso_Link.STL; visual mesh filename=../meshes/D457_in_torso_Link.STL
- added link head_pitch_Link, mass 1.672; collision mesh filename=../meshes/ultra_head_pitch_Link.STL; visual mesh filename=../meshes/ultra_head_pitch_Link.STL
- added link head_yaw_Link, mass 0.8; collision mesh filename=../meshes/head_yaw_Link.STL; visual mesh filename=../meshes/head_yaw_Link.STL
- added link imu_in_pelvis_Link, mass 0.02; collision mesh filename=../meshes/imu_in_pelvis_Link.STL; visual mesh filename=../meshes/imu_in_pelvis_Link.STL
- added link imu_in_torso_Link, mass 0.02; collision mesh filename=../meshes/imu_in_torso_Link.STL; visual mesh filename=../meshes/imu_in_torso_Link.STL
- added link left_ankle_pitch_Link, mass 0.10100813; collision mesh filename=../meshes/left_ankle_pitch_Link.STL; visual mesh filename=../meshes/left_ankle_pitch_Link.STL
- added link left_ankle_roll_Link, mass 0.82544987; collision mesh filename=../meshes/left_ankle_roll_Link.STL; visual mesh filename=../meshes/left_ankle_roll_Link.STL
- added link left_elbow_Link, mass 0.71204442; collision mesh filename=../meshes/left_elbow_Link.STL; visual mesh filename=../meshes/left_elbow_Link.STL
- added link left_hand_palm_Link, mass 0.45864557; collision mesh filename=../meshes/left_hand_palm_Link.STL; visual mesh filename=../meshes/left_hand_palm_Link.STL
- added link left_hip_pitch_Link, mass 1.87345917; collision mesh filename=../meshes/left_hip_pitch_Link.STL; visual mesh filename=../meshes/left_hip_pitch_Link.STL
- added link left_hip_roll_Link, mass 0.74493005; collision mesh filename=../meshes/left_hip_roll_Link.STL; visual mesh filename=../meshes/left_hip_roll_Link.STL
- added link left_hip_yaw_Link, mass 2.64563497; collision mesh filename=../meshes/left_hip_yaw_Link.STL; visual mesh filename=../meshes/left_hip_yaw_Link.STL
- added link left_knee_Link, mass 5.23624455; collision mesh filename=../meshes/left_knee_Link.STL; visual mesh filename=../meshes/left_knee_Link.STL
- added link left_knee_shell_Link, mass 0; collision mesh filename=../meshes/left_knee_shell_Link.STL; visual mesh filename=../meshes/left_knee_shell_Link.STL
- added link left_shoulder_pitch_Link, mass 1.01944747; collision mesh filename=../meshes/left_shoulder_pitch_Link.STL; visual mesh filename=../meshes/left_shoulder_pitch_Link.STL
- added link left_shoulder_roll_Link, mass 0.95854774; collision mesh filename=../meshes/left_shoulder_roll_Link.STL; visual mesh filename=../meshes/left_shoulder_roll_Link.STL
- added link left_shoulder_yaw_Link, mass 0.99955871; collision mesh filename=../meshes/left_shoulder_yaw_Link.STL; visual mesh filename=../meshes/left_shoulder_yaw_Link.STL
- added link left_wrist_pitch_Link, mass 0.56746364; collision mesh filename=../meshes/left_wrist_pitch_Link.STL; visual mesh filename=../meshes/left_wrist_pitch_Link.STL
- added link left_wrist_roll_Link, mass 0.19185994; collision mesh filename=../meshes/left_wrist_roll_Link.STL; visual mesh filename=../meshes/left_wrist_roll_Link.STL
- added link left_wrist_yaw_Link, mass 0.08067756; collision mesh filename=../meshes/left_wrist_yaw_Link.STL; visual mesh filename=../meshes/left_wrist_yaw_Link.STL
- added link pelvis_link, mass 4.98224861; collision mesh filename=../meshes/pelvis_link.STL; visual mesh filename=../meshes/pelvis_link.STL
- added link right_ankle_pitch_Link, mass 0.10100813; collision mesh filename=../meshes/right_ankle_pitch_Link.STL; visual mesh filename=../meshes/right_ankle_pitch_Link.STL
- added link right_ankle_roll_Link, mass 0.82544987; collision mesh filename=../meshes/right_ankle_roll_Link.STL; visual mesh filename=../meshes/right_ankle_roll_Link.STL
- added link right_elbow_Link, mass 0.71187773; collision mesh filename=../meshes/right_elbow_Link.STL; visual mesh filename=../meshes/right_elbow_Link.STL
- added link right_hand_palm_Link, mass 0.45853876; collision mesh filename=../meshes/right_hand_palm_Link.STL; visual mesh filename=../meshes/right_hand_palm_Link.STL
- added link right_hip_pitch_Link, mass 1.87346368; collision mesh filename=../meshes/right_hip_pitch_Link.STL; visual mesh filename=../meshes/right_hip_pitch_Link.STL
- added link right_hip_roll_Link, mass 0.74491385; collision mesh filename=../meshes/right_hip_roll_Link.STL; visual mesh filename=../meshes/right_hip_roll_Link.STL
- added link right_hip_yaw_Link, mass 2.6488815; collision mesh filename=../meshes/right_hip_yaw_Link.STL; visual mesh filename=../meshes/right_hip_yaw_Link.STL
- added link right_knee_Link, mass 5.23155146; collision mesh filename=../meshes/right_knee_Link.STL; visual mesh filename=../meshes/right_knee_Link.STL
- added link right_knee_shell_Link, mass 0; collision mesh filename=../meshes/right_knee_shell_Link.STL; visual mesh filename=../meshes/right_knee_shell_Link.STL
- added link right_shoulder_pitch_Link, mass 1.0194192; collision mesh filename=../meshes/right_shoulder_pitch_Link.STL; visual mesh filename=../meshes/right_shoulder_pitch_Link.STL
- added link right_shoulder_roll_Link, mass 0.95852346; collision mesh filename=../meshes/right_shoulder_roll_Link.STL; visual mesh filename=../meshes/right_shoulder_roll_Link.STL
- added link right_shoulder_yaw_Link, mass 0.99859942; collision mesh filename=../meshes/right_shoulder_yaw_Link.STL; visual mesh filename=../meshes/right_shoulder_yaw_Link.STL
- added link right_wrist_pitch_Link, mass 0.56746364; collision mesh filename=../meshes/right_wrist_pitch_Link.STL; visual mesh filename=../meshes/right_wrist_pitch_Link.STL
- added link right_wrist_roll_Link, mass 0.19185994; collision mesh filename=../meshes/right_wrist_roll_Link.STL; visual mesh filename=../meshes/right_wrist_roll_Link.STL
- added link right_wrist_yaw_Link, mass 0.08067756; collision mesh filename=../meshes/right_wrist_yaw_Link.STL; visual mesh filename=../meshes/right_wrist_yaw_Link.STL
- added link senyun_in_torso_Link, mass 0; collision mesh filename=../meshes/senyun_in_torso_Link.STL; visual mesh filename=../meshes/senyun_in_torso_Link.STL
- added link torso_Link, mass 19.47561404; collision mesh filename=../meshes/torso_Link.STL; visual mesh filename=../meshes/torso_Link.STL
- added link torso_shell_Link, mass 0; collision mesh filename=../meshes/torso_shell_Link.STL; visual mesh filename=../meshes/torso_shell_Link.STL
- added link ultra_head_fisheye_camera_back_Link, mass 0; collision mesh filename=../meshes/ultra_head_fisheye_camera_back_Link.STL; visual mesh filename=../meshes/ultra_head_fisheye_camera_back_Link.STL
- added link ultra_head_fisheye_camera_left_Link, mass 0; collision mesh filename=../meshes/ultra_head_fisheye_camera_left_Link.STL; visual mesh filename=../meshes/ultra_head_fisheye_camera_left_Link.STL
- added link ultra_head_fisheye_camera_right_Link, mass 0; collision mesh filename=../meshes/ultra_head_fisheye_camera_right_Link.STL; visual mesh filename=../meshes/ultra_head_fisheye_camera_right_Link.STL
- added link ultra_head_mid360_Link, mass 0; collision mesh filename=../meshes/ultra_head_mid360_Link.STL; visual mesh filename=../meshes/ultra_head_mid360_Link.STL
- added link ultra_head_stereo_camera_Link, mass 0; collision mesh filename=../meshes/ultra_head_stereo_camera_Link.STL; visual mesh filename=../meshes/ultra_head_stereo_camera_Link.STL
- added link waist_roll_Link, mass 0.13538217; collision mesh filename=../meshes/waist_roll_Link.STL; visual mesh filename=../meshes/waist_roll_Link.STL
- added link waist_yaw_Link, mass 0.24519419; collision mesh filename=../meshes/waist_yaw_Link.STL; visual mesh filename=../meshes/waist_yaw_Link.STL
Joints:
- removed joint left_hand_joint
- removed joint right_hand_joint
- removed joint torso_joint
- added joint D415_in_torso_joint: type fixed, parent torso_Link, child D415_in_torso_Link, origin xyz=0.124480946106383 0 -0.0322504622882431 rpy=0 1.13446401379144 0
- added joint D457_in_torso_joint: type fixed, parent torso_Link, child D457_in_torso_Link, origin xyz=0.148942365217947 4.25892808163051E-05 0.215260754924945 rpy=0 0.698131739779724 0
- added joint left_hand_palm_joint: type fixed, parent left_wrist_yaw_Link, child left_hand_palm_Link, origin xyz=0 0 0 rpy=0 0 0
- added joint left_knee_shell_joint: type fixed, parent left_knee_Link, child left_knee_shell_Link, origin xyz=0 0 0 rpy=0 0 0
- added joint right_hand_palm_joint: type fixed, parent right_wrist_yaw_Link, child right_hand_palm_Link, origin xyz=0 0 0 rpy=0 0 0
- added joint right_knee_shell_joint: type fixed, parent right_knee_Link, child right_knee_shell_Link, origin xyz=0 0 0 rpy=0 0 0
- added joint senyun_in_torso_joint: type fixed, parent torso_Link, child senyun_in_torso_Link, origin xyz=0.0302999999991496 -0.137203916977493 0.187745894474438 rpy=0.226892802759255 0 0
- added joint torso_shell_joint: type fixed, parent torso_Link, child torso_shell_Link, origin xyz=0 0 0 rpy=0 0 0
- added joint ultra_head_fisheye_camera_back_joint: type fixed, parent head_pitch_Link, child ultra_head_fisheye_camera_back_Link, origin xyz=-0.078845195202418 0 0.0384247314841796 rpy=0 -0.133379281154304 0
- added joint ultra_head_fisheye_camera_left_joint: type fixed, parent head_pitch_Link, child ultra_head_fisheye_camera_left_Link, origin xyz=0.0150035360841172 0.07489976194252 0.0297028705940667 rpy=-0.0514108672262889 -0.0188992743027947 -0.0437102135661861
- added joint ultra_head_fisheye_camera_right_joint: type fixed, parent head_pitch_Link, child ultra_head_fisheye_camera_right_Link, origin xyz=0.0150035360639564 -0.0748997619425288 0.0297028706040139 rpy=0.0514116929184328 -0.0197300914132888 0.0436674542870696
- added joint ultra_head_mid360_joint: type fixed, parent head_yaw_Link, child ultra_head_mid360_Link, origin xyz=0.0199258874260123 0 0.137544948520896 rpy=0 0 0
- added joint ultra_head_stereo_camera_joint: type fixed, parent head_pitch_Link, child ultra_head_stereo_camera_Link, origin xyz=0.0919825582208656 0 -0.0302207411626506 rpy=0 0.241209429948845 0
- joint head_pitch_joint: axis 0 1 0 -> 0.0 1.0 0.0; child head_pitch_link -> head_pitch_Link; limit lower=-0.43633 upper=0.26180 effort=0 velocity=0 -> lower=-0.4363323129985824 upper=0.2617993877991494 effort=6 velocity=12.775810124598491; origin (none) -> xyz=0 0 0.230630601825014 rpy=0 0 0; parent head_yaw_link -> head_yaw_Link
- joint head_yaw_joint: axis 0 0 1 -> 0.0 0.0 1.0; child head_yaw_link -> head_yaw_Link; limit lower=-1.570796 upper=1.570796 effort=0 velocity=0 -> lower=-1.0471975511965976 upper=1.0471975511965976 effort=6 velocity=12.775810124598491; origin (none) -> xyz=0.030299999999954 0 0.288960095038301 rpy=0 0 0; parent torso -> torso_Link
- joint imu_in_pelvis_joint: child imu_in_pelvis_link -> imu_in_pelvis_Link; origin (none) -> xyz=0.00437000000055574 0 -0.211649999998792 rpy=0 0 0; parent pelvis -> pelvis_link
- joint imu_in_torso_joint: child imu_in_torso_link -> imu_in_torso_Link; origin (none) -> xyz=0 0 0.111850000001117 rpy=0 0 0; parent torso -> torso_Link
- joint left_ankle_pitch_joint: axis 0 1 0 -> 0.0 1.0 0.0; child left_ankle_pitch_link -> left_ankle_pitch_Link; limit lower=-0.907571 upper=0.523599 effort=0 velocity=0 -> lower=-0.9075712110370514 upper=0.5235987755982988 effort=118.2 velocity=10.8; origin (none) -> xyz=0 0.00150000000138217 -0.414999999999997 rpy=0 0 0; parent left_knee_link -> left_knee_Link
- joint left_ankle_roll_joint: axis 1 0 0 -> 1.0 0.0 0.0; child left_foot -> left_ankle_roll_Link; limit lower=-0.349066 upper=0.349066 effort=0 velocity=0 -> lower=-0.3490658503988659 upper=0.3490658503988659 effort=54.75 velocity=19.37; origin (none) -> xyz=0 0 0 rpy=0 0 0; parent left_ankle_pitch_link -> left_ankle_pitch_Link
- joint left_elbow_joint: axis 0 1 0 -> 0.0 1.0 0.0; child left_elbow_link -> left_elbow_Link; limit lower=-0.959931 upper=1.745329 effort=0 velocity=4 -> lower=-0.9599310885968813 upper=1.7453292519943295 effort=24 velocity=15.707963267948966; origin (none) -> xyz=0.01 0 -0.1325 rpy=0 0 0; parent left_shoulder_yaw_link -> left_shoulder_yaw_Link
- joint left_hip_pitch_joint: axis 0 1 0 -> 0.0 1.0 0.0; child left_hip_pitch_link -> left_hip_pitch_Link; limit lower=-2.932153 upper=2.687807 effort=0 velocity=0 -> lower=-2.5132741228718345 upper=2.9321531433504737 effort=220 velocity=12.042771838760874; origin (none) -> xyz=0 0.122982962907307 -0.178753185592275 rpy=-0.261799387796752 0 0; parent pelvis -> pelvis_link
- joint left_hip_roll_joint: axis 1 0 0 -> 1.0 0.0 0.0; child left_hip_roll_link -> left_hip_roll_Link; limit lower=-1.047198 upper=1.745329 effort=0 velocity=0 -> lower=-0.5235987755982988 upper=1.4835298641951802 effort=220 velocity=12.042771838760874; origin (none) -> xyz=0 0.0113162873210235 -0.0422329592212282 rpy=0.261799387796752 0 0; parent left_hip_pitch_link -> left_hip_pitch_Link
- joint left_hip_yaw_joint: axis 0 0 1 -> 0.0 0.0 1.0; child left_hip_yaw_link -> left_hip_yaw_Link; limit lower=-2.757620 upper=2.757620 effort=0 velocity=0 -> lower=-2.722713633111154 upper=2.722713633111154 effort=220 velocity=12.042771838760874; origin (none) -> xyz=0 0 0 rpy=0 0 0; parent left_hip_roll_link -> left_hip_roll_Link
- joint left_index_bent_1: limit lower=0 upper=4096 effort=0 velocity=0 -> lower=0 upper=1.5708 effort=0 velocity=0; origin (none) -> xyz=0 0.025 0
- joint left_index_wiggles_0: limit lower=0 upper=4096 effort=0 velocity=0 -> lower=0 upper=1.5708 effort=0 velocity=0; origin (none) -> xyz=0 0.04 0.02; parent left_hand_link -> left_hand_palm_Link
- joint left_knee_joint: axis 0 1 0 -> 0.0 1.0 0.0; child left_knee_link -> left_knee_Link; limit lower=-0.174533 upper=2.583087 effort=0 velocity=0 -> lower=-0.12217304763960307 upper=2.530727415391778 effort=320 velocity=14.660765716752367; origin (none) -> xyz=0 0 -0.369999999999994 rpy=0 0 0; parent left_hip_yaw_link -> left_hip_yaw_Link
- joint left_middle_bent: limit lower=0 upper=4096 effort=0 velocity=0 -> lower=0 upper=1.5708 effort=0 velocity=0; origin (none) -> xyz=0 0.04 0; parent left_hand_link -> left_hand_palm_Link
- joint left_pinky_bent_1: limit lower=0 upper=4096 effort=0 velocity=0 -> lower=0 upper=1.5708 effort=0 velocity=0; origin (none) -> xyz=0 0.025 0
- joint left_pinky_wiggles_0: limit lower=0 upper=4096 effort=0 velocity=0 -> lower=0 upper=1.5708 effort=0 velocity=0; origin (none) -> xyz=0 0.04 -0.04; parent left_hand_link -> left_hand_palm_Link
- joint left_ring_bent_1: limit lower=0 upper=4096 effort=0 velocity=0 -> lower=0 upper=1.5708 effort=0 velocity=0; origin (none) -> xyz=0 0.025 0
- joint left_ring_wiggles_0: limit lower=0 upper=4096 effort=0 velocity=0 -> lower=0 upper=1.5708 effort=0 velocity=0; origin (none) -> xyz=0 0.04 -0.02; parent left_hand_link -> left_hand_palm_Link
- joint left_shoulder_pitch_joint: axis 0 1 0 -> 0.0 1.0 0.0; child left_shoulder_pitch_link -> left_shoulder_pitch_Link; limit lower=-2.879793 upper=2.879793 effort=0 velocity=4 -> lower=-2.8797932657906435 upper=2.8797932657906435 effort=60 velocity=13.613568165555769; origin (none) -> xyz=0.03029999999793 0.148224512812617 0.283817906204843 rpy=0.0872664625997163 0 0; parent torso -> torso_Link
- joint left_shoulder_roll_joint: axis 0 0 1 -> 1.0 0.0 0.0; child left_shoulder_roll_link -> left_shoulder_roll_Link; limit lower=-0.087266 upper=2.617994 effort=0 velocity=4 -> lower=-0.08726646259971647 upper=2.6179938779914944 effort=60 velocity=13.613568165555769; origin (none) -> xyz=0 0.0590000000000002 0 rpy=-0.0872664625997163 0 0; parent left_shoulder_pitch_link -> left_shoulder_pitch_Link
- joint left_shoulder_yaw_joint: axis 1 0 0 -> 0.0 0.0 1.0; child left_shoulder_yaw_link -> left_shoulder_yaw_Link; limit lower=-2.792527 upper=2.792527 effort=0 velocity=4 -> lower=-2.792526803190927 upper=2.792526803190927 effort=24 velocity=15.707963267948966; origin (none) -> xyz=0 0.0100000000000015 -0.14749999999002 rpy=0 0 0; parent left_shoulder_roll_link -> left_shoulder_roll_Link
- joint left_thumb_bent_2: limit lower=0 upper=4096 effort=0 velocity=0 -> lower=0 upper=1.5708 effort=0 velocity=0; origin (none) -> xyz=0 0.025 0
- joint left_thumb_roration_0: limit lower=0 upper=4096 effort=0 velocity=0 -> lower=0 upper=1.5708 effort=0 velocity=0; origin (none) -> xyz=0 0.03 0; parent left_hand_link -> left_hand_palm_Link
- joint left_thumb_wiggles_1: limit lower=0 upper=4096 effort=0 velocity=0 -> lower=0 upper=1.5708 effort=0 velocity=0; origin (none) -> xyz=0 0.025 0
- joint left_wrist_pitch_joint: axis 0 1 0 -> 0.0 1.0 0.0; child left_wrist_pitch_link -> left_wrist_pitch_Link; limit lower=-1.623156 upper=1.623156 effort=0 velocity=4 -> lower=-1.6231562043547265 upper=1.6231562043547265 effort=6 velocity=12.775810124598491; origin (none) -> xyz=0.0600000000000002 0 0 rpy=0 0 0; parent left_wrist_roll_link -> left_wrist_roll_Link
- joint left_wrist_roll_joint: axis 1 0 0 -> 1.0 0.0 0.0; child left_wrist_roll_link -> left_wrist_roll_Link; limit lower=-2.792527 upper=2.792527 effort=0 velocity=4 -> lower=-2.792526803190927 upper=2.792526803190927 effort=24 velocity=15.707963267948966; origin (none) -> xyz=0.129 0 -0.00999999999999995 rpy=0 0 0; parent left_elbow_link -> left_elbow_Link
- joint left_wrist_yaw_joint: axis 0 0 1 -> 0.0 0.0 1.0; child left_wrist_yaw_link -> left_wrist_yaw_Link; limit lower=-1.623156 upper=1.623156 effort=0 velocity=4 -> lower=-1.6231562043547265 upper=1.6231562043547265 effort=6 velocity=12.775810124598491; origin (none) -> xyz=0.046 0 0 rpy=0 0 0; parent left_wrist_pitch_link -> left_wrist_pitch_Link
- joint right_ankle_pitch_joint: axis 0 1 0 -> 0.0 1.0 0.0; child right_ankle_pitch_link -> right_ankle_pitch_Link; limit lower=-0.907571 upper=0.523599 effort=0 velocity=0 -> lower=-0.9075712110370514 upper=0.5235987755982988 effort=118.2 velocity=10.8; origin (none) -> xyz=0 -0.001499999998404 -0.415000000000001 rpy=0 0 0; parent right_knee_link -> right_knee_Link
- joint right_ankle_roll_joint: axis 1 0 0 -> 1.0 0.0 0.0; child right_foot -> right_ankle_roll_Link; limit lower=-0.349066 upper=0.349066 effort=0 velocity=0 -> lower=-0.3490658503988659 upper=0.3490658503988659 effort=54.75 velocity=19.37; origin (none) -> xyz=0 0 0 rpy=0 0 0; parent right_ankle_pitch_link -> right_ankle_pitch_Link
- joint right_elbow_joint: axis 0 1 0 -> 0.0 1.0 0.0; child right_elbow_link -> right_elbow_Link; limit lower=-0.959931 upper=1.745329 effort=0 velocity=4 -> lower=-0.9599310885968813 upper=1.7453292519943295 effort=24 velocity=15.707963267948966; origin (none) -> xyz=0.00999999997356363 0 -0.132999999990091 rpy=0 0 0; parent right_shoulder_yaw_link -> right_shoulder_yaw_Link
- joint right_hip_pitch_joint: axis 0 1 0 -> 0.0 1.0 0.0; child right_hip_pitch_link -> right_hip_pitch_Link; limit lower=-2.932153 upper=2.687807 effort=0 velocity=0 -> lower=-2.5132741228718345 upper=2.9321531433504737 effort=220 velocity=12.042771838760874; origin (none) -> xyz=0 -0.122982962906483 -0.178753185592622 rpy=0.261799387800366 0 0; parent pelvis -> pelvis_link
- joint right_hip_roll_joint: axis 1 0 0 -> 1.0 0.0 0.0; child right_hip_roll_link -> right_hip_roll_Link; limit lower=-1.047198 upper=1.745329 effort=0 velocity=0 -> lower=-1.4835298641951802 upper=0.5235987755982988 effort=220 velocity=12.042771838760874; origin (none) -> xyz=-0.00109999056710738 -0.0113162873211849 -0.042232959221232 rpy=-0.261799387800366 0 0; parent right_hip_pitch_link -> right_hip_pitch_Link
- joint right_hip_yaw_joint: axis 0 0 1 -> 0.0 0.0 1.0; child right_hip_yaw_link -> right_hip_yaw_Link; limit lower=-2.757620 upper=2.757620 effort=0 velocity=0 -> lower=-2.722713633111154 upper=2.722713633111154 effort=220 velocity=12.042771838760874; origin (none) -> xyz=0 0 0 rpy=0 0 0; parent right_hip_roll_link -> right_hip_roll_Link
- joint right_index_bent_1: limit lower=0 upper=4096 effort=0 velocity=0 -> lower=0 upper=1.5708 effort=0 velocity=0; origin (none) -> xyz=0 0.025 0
- joint right_index_wiggles_0: limit lower=0 upper=4096 effort=0 velocity=0 -> lower=0 upper=1.5708 effort=0 velocity=0; origin (none) -> xyz=0 0.04 0.02; parent right_hand_link -> right_hand_palm_Link
- joint right_knee_joint: axis 0 1 0 -> 0.0 1.0 0.0; child right_knee_link -> right_knee_Link; limit lower=-0.174533 upper=2.583087 effort=0 velocity=0 -> lower=-0.12217304763960307 upper=2.530727415391778 effort=320 velocity=14.660765716752367; origin (none) -> xyz=0 0 -0.369999999999993 rpy=0 0 0; parent right_hip_yaw_link -> right_hip_yaw_Link
- joint right_middle_bent: limit lower=0 upper=4096 effort=0 velocity=0 -> lower=0 upper=1.5708 effort=0 velocity=0; origin (none) -> xyz=0 0.04 0; parent right_hand_link -> right_hand_palm_Link
- joint right_pinky_bent_1: limit lower=0 upper=4096 effort=0 velocity=0 -> lower=0 upper=1.5708 effort=0 velocity=0; origin (none) -> xyz=0 0.025 0
- joint right_pinky_wiggles_0: limit lower=0 upper=4096 effort=0 velocity=0 -> lower=0 upper=1.5708 effort=0 velocity=0; origin (none) -> xyz=0 0.04 -0.04; parent right_hand_link -> right_hand_palm_Link
- joint right_ring_bent_1: limit lower=0 upper=4096 effort=0 velocity=0 -> lower=0 upper=1.5708 effort=0 velocity=0; origin (none) -> xyz=0 0.025 0
- joint right_ring_wiggles_0: limit lower=0 upper=4096 effort=0 velocity=0 -> lower=0 upper=1.5708 effort=0 velocity=0; origin (none) -> xyz=0 0.04 -0.02; parent right_hand_link -> right_hand_palm_Link
- joint right_shoulder_pitch_joint: axis 0 1 0 -> 0.0 1.0 0.0; child right_shoulder_pitch_link -> right_shoulder_pitch_Link; limit lower=-2.879793 upper=2.879793 effort=0 velocity=4 -> lower=-2.8797932657906404 upper=2.8797932657906435 effort=60 velocity=13.613568165555769; origin (none) -> xyz=0.03030000000207 -0.148224512812557 0.283817906204843 rpy=-0.0872664625997163 0 0; parent torso -> torso_Link
- joint right_shoulder_roll_joint: axis 0 0 1 -> 1.0 0.0 0.0; child right_shoulder_roll_link -> right_shoulder_roll_Link; limit lower=-2.617994 upper=0.087266 effort=0 velocity=4 -> lower=-2.6179938779914944 upper=0.08726646259971647 effort=60 velocity=13.613568165555769; origin (none) -> xyz=0 -0.0589999999982601 0 rpy=0.0872664625997163 0 0; parent right_shoulder_pitch_link -> right_shoulder_pitch_Link
- joint right_shoulder_yaw_joint: axis 1 0 0 -> 0.0 0.0 1.0; child right_shoulder_yaw_link -> right_shoulder_yaw_Link; limit lower=-2.792527 upper=2.792527 effort=0 velocity=4 -> lower=-2.792526803190927 upper=2.792526803190927 effort=24 velocity=15.707963267948966; origin (none) -> xyz=0 -0.0100000000003387 -0.147499999999977 rpy=0 0 0; parent right_shoulder_roll_link -> right_shoulder_roll_Link
- joint right_thumb_bent_2: limit lower=0 upper=4096 effort=0 velocity=0 -> lower=0 upper=1.5708 effort=0 velocity=0; origin (none) -> xyz=0 0.025 0
- joint right_thumb_rotation_0: limit lower=0 upper=4096 effort=0 velocity=0 -> lower=0 upper=1.5708 effort=0 velocity=0; origin (none) -> xyz=0 0.03 0; parent right_hand_link -> right_hand_palm_Link
- joint right_thumb_wiggles_1: limit lower=0 upper=4096 effort=0 velocity=0 -> lower=0 upper=1.5708 effort=0 velocity=0; origin (none) -> xyz=0 0.025 0
- joint right_wrist_pitch_joint: axis 0 1 0 -> 0.0 1.0 0.0; child right_wrist_pitch_link -> right_wrist_pitch_Link; limit lower=-1.623156 upper=1.623156 effort=0 velocity=4 -> lower=-1.6231562043547265 upper=1.6231562043547265 effort=6 velocity=12.775810124598491; origin (none) -> xyz=0.0600000000000003 0 0 rpy=0 0 0; parent right_wrist_roll_link -> right_wrist_roll_Link
- joint right_wrist_roll_joint: axis 1 0 0 -> 1.0 0.0 0.0; child right_wrist_roll_link -> right_wrist_roll_Link; limit lower=-2.792527 upper=2.792527 effort=0 velocity=4 -> lower=-2.792526803190927 upper=2.792526803190927 effort=24 velocity=15.707963267948966; origin (none) -> xyz=0.129 0 -0.00999999999980283 rpy=0 0 0; parent right_elbow_link -> right_elbow_Link
- joint right_wrist_yaw_joint: axis 0 0 1 -> 0.0 0.0 1.0; child right_wrist_yaw_link -> right_wrist_yaw_Link; limit lower=-1.623156 upper=1.623156 effort=0 velocity=4 -> lower=-1.6231562043547265 upper=1.6231562043547265 effort=6 velocity=12.775810124598491; origin (none) -> xyz=0.046 0 0 rpy=0 0 0; parent right_wrist_pitch_link -> right_wrist_pitch_Link
- joint waist_pitch_joint: axis 0 1 0 -> 0.0 1.0 0.0; child waist_pitch_link -> torso_Link; limit lower=-0.523599 upper=0.523599 effort=0 velocity=0 -> lower=-0.4886921905584123 upper=0.4188790204786391 effort=118 velocity=9.24785; origin (none) -> xyz=-0.0199999999998296 0 0.00500000000000012 rpy=0 0 0; parent waist_yaw_link -> waist_roll_Link
- joint waist_roll_joint: axis 1 0 0 -> 1.0 0.0 0.0; child waist_roll_link -> waist_roll_Link; limit lower=-0.349066 upper=0.349066 effort=0 velocity=0 -> lower=-0.3490658503988659 upper=0.3490658503988659 effort=46 velocity=22.7; origin (none) -> xyz=0 0 0 rpy=0 0 0; parent pelvis -> waist_yaw_Link
- joint waist_yaw_joint: axis 0 0 1 -> 0.0 0.0 1.0; child waist_yaw_link -> waist_yaw_Link; limit lower=-2.617994 upper=2.617994 effort=0 velocity=0 -> lower=-2.6179938779914944 upper=2.6179938779914944 effort=220 velocity=12.042771838760874; origin (none) -> xyz=0 0 0 rpy=0 0 0; parent waist_roll_link -> pelvis_link
