Commit message: Align A3 skeleton feedback and omit unavailable wrist cameras

File: agibot/A3/resource/a3_ultra.urdf (robot description, URDF)
Before this commit: robot A3_ULTRA_T2D5, 67 links, 66 joints
Links:
- added link left_index_tip
- added link left_middle_tip
- added link left_pinky_tip
- added link left_ring_tip
- added link left_thumb_tip
- added link right_index_tip
- added link right_middle_tip
- added link right_pinky_tip
- added link right_ring_tip
- added link right_thumb_tip
Joints:
- added joint left_index_tip_fixed: type fixed, parent left_hand_channel_4, child left_index_tip, origin xyz=0.03 0 0
- added joint left_middle_tip_fixed: type fixed, parent left_hand_channel_5, child left_middle_tip, origin xyz=0.035 0 0
- added joint left_pinky_tip_fixed: type fixed, parent left_hand_channel_9, child left_pinky_tip, origin xyz=0.025 0 0
- added joint left_ring_tip_fixed: type fixed, parent left_hand_channel_7, child left_ring_tip, origin xyz=0.03 0 0
- added joint left_thumb_tip_fixed: type fixed, parent left_hand_channel_2, child left_thumb_tip, origin xyz=0.025 0 0
- added joint right_index_tip_fixed: type fixed, parent right_hand_channel_4, child right_index_tip, origin xyz=0.03 0 0
- added joint right_middle_tip_fixed: type fixed, parent right_hand_channel_5, child right_middle_tip, origin xyz=0.035 0 0
- added joint right_pinky_tip_fixed: type fixed, parent right_hand_channel_9, child right_pinky_tip, origin xyz=0.025 0 0
- added joint right_ring_tip_fixed: type fixed, parent right_hand_channel_7, child right_ring_tip, origin xyz=0.03 0 0
- added joint right_thumb_tip_fixed: type fixed, parent right_hand_channel_2, child right_thumb_tip, origin xyz=0.025 0 0
- joint left_hand_palm_joint: origin xyz=0 0 0 rpy=0 0 0 -> xyz=0.08 0 0 rpy=0 0 0
- joint left_index_bent_1: origin xyz=0 0.025 0 -> xyz=0.035 0 0
- joint left_index_wiggles_0: origin xyz=0 0.04 0.02 -> xyz=0.055 0.024 0.008
- joint left_middle_bent: origin xyz=0 0.04 0 -> xyz=0.07 0.008 0.01
- joint left_pinky_bent_1: origin xyz=0 0.025 0 -> xyz=0.03 0 0
- joint left_pinky_wiggles_0: origin xyz=0 0.04 -0.04 -> xyz=0.045 -0.028 0.006
- joint left_ring_bent_1: origin xyz=0 0.025 0 -> xyz=0.035 0 0
- joint left_ring_wiggles_0: origin xyz=0 0.04 -0.02 -> xyz=0.055 -0.01 0.008
- joint left_thumb_bent_2: origin xyz=0 0.025 0 -> xyz=0.025 0 0
- joint left_thumb_roration_0: origin xyz=0 0.03 0 -> xyz=0.025 0.034 0.006
- joint left_thumb_wiggles_1: origin xyz=0 0.025 0 -> xyz=0.025 0 0
- joint right_hand_palm_joint: origin xyz=0 0 0 rpy=0 0 0 -> xyz=0.08 0 0 rpy=0 0 0
- joint right_index_bent_1: origin xyz=0 0.025 0 -> xyz=0.035 0 0
- joint right_index_wiggles_0: origin xyz=0 0.04 0.02 -> xyz=0.055 0.024 0.008
- joint right_middle_bent: origin xyz=0 0.04 0 -> xyz=0.07 0.008 0.01
- joint right_pinky_bent_1: origin xyz=0 0.025 0 -> xyz=0.03 0 0
- joint right_pinky_wiggles_0: origin xyz=0 0.04 -0.04 -> xyz=0.045 -0.028 0.006
- joint right_ring_bent_1: origin xyz=0 0.025 0 -> xyz=0.035 0 0
- joint right_ring_wiggles_0: origin xyz=0 0.04 -0.02 -> xyz=0.055 -0.01 0.008
- joint right_thumb_bent_2: origin xyz=0 0.025 0 -> xyz=0.025 0 0
- joint right_thumb_rotation_0: origin xyz=0 0.03 0 -> xyz=0.025 0.034 0.006
- joint right_thumb_wiggles_1: origin xyz=0 0.025 0 -> xyz=0.025 0 0

Commit message: fix: route official A3 audio and hand feedback

File: agibot/A3/resource/a3_ultra.urdf (robot description, URDF)
Before this commit: robot A3_ULTRA_T2D5, 77 links, 76 joints
Joints:
- removed joint left_thumb_roration_0
- added joint left_thumb_rotation_0: type revolute, parent left_hand_palm_Link, child left_hand_channel_0, origin xyz=0.025 0.034 0.006, axis 1 0 0, limit lower=0 upper=1.5708 effort=0 velocity=0

Commit message: fix: restore stable A3 media relay baseline

File: agibot/A3/resource/a3_ultra.urdf (robot description, URDF)
Before this commit: robot A3_ULTRA_T2D5, 77 links, 76 joints
Joints:
- removed joint left_thumb_rotation_0
- added joint left_thumb_roration_0: type revolute, parent left_hand_palm_Link, child left_hand_channel_0, origin xyz=0.025 0.034 0.006, axis 1 0 0, limit lower=0 upper=1.5708 effort=0 velocity=0

Commit message: fix: use calibrated O10 hand kinematics for A3

File: agibot/A3/resource/a3_ultra.urdf (robot description, URDF)
Before this commit: robot A3_ULTRA_T2D5, 77 links, 76 joints
Joints:
- removed joint left_hand_palm_joint
- removed joint right_hand_palm_joint
- added joint left_hand_O10_joint: type fixed, parent left_wrist_yaw_Link, child left_hand_palm_Link, origin xyz=0.08 0 0 rpy=3.14 0 -1.57
- added joint right_hand_O10_joint: type fixed, parent right_wrist_yaw_Link, child right_hand_palm_Link, origin xyz=0.08 0 0 rpy=-3.14 0 1.5708
