Commit message: fix: validate A3 host relay image dependencies

File: agibot/A3/resource/a3_o10_hand.urdf (robot description, URDF)
Before this commit: robot A3_O10_HANDS, 46 links, 46 joints
Joints:
- joint L_palm_joint: origin xyz=0 0 0 rpy=1.5707963 0 0 -> xyz=0 0 0 rpy=0 1.5707963 0
- joint R_palm_joint: origin xyz=0 0 0 rpy=-1.5707963 0 0 -> xyz=0 0 0 rpy=0 1.5707963 0

Commit message: fix: align A3 O10 hand pose and feedback signs

File: agibot/A3/resource/a3_o10_hand.urdf (robot description, URDF)
Before this commit: robot A3_O10_HANDS, 46 links, 46 joints
Joints:
- joint L_palm_joint: origin xyz=0 0 0 rpy=0 1.5707963 0 -> xyz=0 0 0 rpy=0 1.5707963 -1.5707963
- joint R_palm_joint: origin xyz=0 0 0 rpy=0 1.5707963 0 -> xyz=0 0 0 rpy=0 1.5707963 1.5707963

Commit message: fix: correct A3 hand pose and relay readiness

File: agibot/A3/resource/a3_o10_hand.urdf (robot description, URDF)
Before this commit: robot A3_O10_HANDS, 46 links, 46 joints
Joints:
- joint L_palm_joint: origin xyz=0 0 0 rpy=0 1.5707963 -1.5707963 -> xyz=0 0 0 rpy=0 1.5707963 0
- joint R_palm_joint: origin xyz=0 0 0 rpy=0 1.5707963 1.5707963 -> xyz=0 0 0 rpy=0 1.5707963 0

Commit message: fix: correct A3 hand frame and state QoS

File: agibot/A3/resource/a3_o10_hand.urdf (robot description, URDF)
Before this commit: robot A3_O10_HANDS, 46 links, 46 joints
Joints:
- joint L_palm_joint: origin xyz=0 0 0 rpy=0 1.5707963 -1.5707963 -> xyz=0 0 0 rpy=-3.1415927 0 1.5707963
- joint R_palm_joint: origin xyz=0 0 0 rpy=0 1.5707963 1.5707963 -> xyz=0 0 0 rpy=-3.1415927 0 -1.5707963

Commit message: fix: remove unused relay dependencies and shared zenoh override

File: agibot/A3/resource/a3_o10_hand.urdf (robot description, URDF)
Before this commit: robot A3_O10_HANDS, 46 links, 46 joints
Joints:
- joint L_palm_joint: origin xyz=0 0 0 rpy=-3.1415927 0 1.5707963 -> xyz=0 0 0 rpy=3.1415914 -0.0015927 1.5715927
- joint R_palm_joint: origin xyz=0 0 0 rpy=-3.1415927 0 -1.5707963 -> xyz=0 0 0 rpy=3.1415926 -0.0015927 -1.5707927

Commit message: fix: calibrate A3 hand pose and state refresh

File: agibot/A3/resource/a3_o10_hand.urdf (robot description, URDF)
Before this commit: robot A3_O10_HANDS, 46 links, 46 joints
Joints:
- joint L_palm_joint: origin xyz=0 0 0 rpy=3.1415914 -0.0015927 1.5715927 -> xyz=0 0 0 rpy=-3.14 0 0.0007964
- joint R_palm_joint: origin xyz=0 0 0 rpy=3.1415926 -0.0015927 -1.5707927 -> xyz=0 0 0 rpy=-0.0015927 0 0.0000037

Commit message: fix: apply final A3 hand orientation correction

File: agibot/A3/resource/a3_o10_hand.urdf (robot description, URDF)
Before this commit: robot A3_O10_HANDS, 46 links, 46 joints
Joints:
- joint L_palm_joint: origin xyz=0 0 0 rpy=-3.14 0 0.0007964 -> xyz=0 0 0 rpy=0.0015927 -2.5e-06 0.0007963
- joint R_palm_joint: origin xyz=0 0 0 rpy=-0.0015927 0 0.0000037 -> xyz=0 0 0 rpy=3.14 0 0.0000036

Commit message: fix: calibrate A3 hand pose and sensor cadence

File: agibot/A3/resource/a3_o10_hand.urdf (robot description, URDF)
Before this commit: robot A3_O10_HANDS, 46 links, 46 joints
Joints:
- joint L_palm_joint: origin xyz=0 0 0 rpy=0.0015927 -2.5e-06 0.0007963 -> xyz=0 0 0 rpy=0.0015927 -0.0000025 0.0007963

Commit message: fix: apply observed hand pose correction

File: agibot/A3/resource/a3_o10_hand.urdf (robot description, URDF)
Before this commit: robot A3_O10_HANDS, 46 links, 46 joints
Joints:
- joint L_palm_joint: origin xyz=0 0 0 rpy=0.0015927 -0.0000025 0.0007963 -> xyz=0 0 0 rpy=-3.1415913 0.0015939 -1.57
- joint R_palm_joint: origin xyz=0 0 0 rpy=3.14 0 0.0000036 -> xyz=0 0 0 rpy=-0.0 -0.0015926 -1.5707926

Commit message: fix: align A3 hands from observed orientation

File: agibot/A3/resource/a3_o10_hand.urdf (robot description, URDF)
Before this commit: robot A3_O10_HANDS, 46 links, 46 joints
Joints:
- joint L_palm_joint: origin xyz=0 0 0 rpy=-3.1415913 0.0015939 -1.57 -> xyz=0 0 0 rpy=1.5707963 0 0.0008
- joint R_palm_joint: origin xyz=0 0 0 rpy=-0.0 -0.0015926 -1.5707926 -> xyz=0 0 0 rpy=1.5707963 0 0.000004

Commit message: fix: correct left and right A3 hand poses

File: agibot/A3/resource/a3_o10_hand.urdf (robot description, URDF)
Before this commit: robot A3_O10_HANDS, 46 links, 46 joints
Joints:
- joint L_palm_joint: origin xyz=0 0 0 rpy=1.5707963 0 0.0008 -> xyz=0 0 0 rpy=-1.5707964 -0.0000025 0.0007927
- joint R_palm_joint: origin xyz=0 0 0 rpy=1.5707963 0 0.000004 -> xyz=0 0 0 rpy=-1.567611 -0.000000001 -3.1415893

Commit message: fix: calibrate A3 hands from latest pose feedback

File: agibot/A3/resource/a3_o10_hand.urdf (robot description, URDF)
Before this commit: robot A3_O10_HANDS, 46 links, 46 joints
Joints:
- joint L_palm_joint: origin xyz=0 0 0 rpy=-1.5707964 -0.0000025 0.0007927 -> xyz=0 0 0 rpy=1.567611 0.0000025 -3.1407927
- joint R_palm_joint: origin xyz=0 0 0 rpy=-1.567611 -0.000000001 -3.1415893 -> xyz=0 0 0 rpy=-1.5707963 0 0.0000034

Commit message: fix: refine A3 hand orientation from feedback

File: agibot/A3/resource/a3_o10_hand.urdf (robot description, URDF)
Before this commit: robot A3_O10_HANDS, 46 links, 46 joints
Joints:
- joint L_palm_joint: origin xyz=0 0 0 rpy=1.567611 0.0000025 -3.1407927 -> xyz=0 0 0 rpy=-1.5739817 0 -3.1408
- joint R_palm_joint: origin xyz=0 0 0 rpy=-1.5707963 0 0.0000034 -> xyz=0 0 0 rpy=1.5739817 0 -3.1415887
