Commit message: fix: 完善山猫S10电池灯光和媒体流

File: deep_robotics/lynx_s10/resource/S10.urdf (robot description, URDF)
Before this commit: robot S10, 20 links, 19 joints
Links:
- link base_link: geometry collision box size=0.16 0.048 0.60; collision cylinder length=0.60 radius=0.08

Commit message: Improve Lynx S10 media streams and light controls

File: deep_robotics/lynx_s10/resource/S10.urdf (robot description, URDF)
Before this commit: robot S10, 20 links, 19 joints
Links:
- added link front_marker_close
- added link front_marker_left
- added link front_marker_right
- added link front_marker_tip
- link base_link: geometry collision box size=0.16 0.048 0.60; collision cylinder length=0.60 radius=0.08
Joints:
- added joint front_marker_close_joint: type fixed, parent front_marker_right, child front_marker_close, origin xyz=0.30 0 0 rpy=0 0 0
- added joint front_marker_left_joint: type fixed, parent front_marker_tip, child front_marker_left, origin xyz=-0.15 0 -0.25 rpy=0 0 0
- added joint front_marker_right_joint: type fixed, parent front_marker_left, child front_marker_right, origin xyz=-0.15 0 0.25 rpy=0 0 0
- added joint front_marker_tip_joint: type fixed, parent base_link, child front_marker_tip, origin xyz=0.42 0 0.18 rpy=0 0 0

Commit message: Fix Lynx S10 light and media forwarding

File: deep_robotics/lynx_s10/resource/S10.urdf (robot description, URDF)
Before this commit: robot S10, 24 links, 23 joints
Joints:
- joint front_marker_close_joint: origin xyz=0.30 0 0 rpy=0 0 0 -> xyz=0.075 0 0 rpy=0 0 0
- joint front_marker_left_joint: origin xyz=-0.15 0 -0.25 rpy=0 0 0 -> xyz=-0.0375 0 -0.0625 rpy=0 0 0
- joint front_marker_right_joint: origin xyz=-0.15 0 0.25 rpy=0 0 0 -> xyz=-0.0375 0 0.0625 rpy=0 0 0
- joint front_marker_tip_joint: origin xyz=0.42 0 0.18 rpy=0 0 0 -> xyz=0.105 0 0.045 rpy=0 0 0

Commit message: fix lynx s10 media forwarding and sensor resources

File: deep_robotics/lynx_s10/resource/S10.urdf (robot description, URDF)
Before this commit: robot S10, 24 links, 23 joints
Joints:
- joint front_marker_close_joint: origin xyz=0.075 0 0 rpy=0 0 0 -> xyz=0.12 0 0 rpy=0 0 0
- joint front_marker_left_joint: origin xyz=-0.0375 0 -0.0625 rpy=0 0 0 -> xyz=-0.06 0 -0.035 rpy=0 0 0
- joint front_marker_right_joint: origin xyz=-0.0375 0 0.0625 rpy=0 0 0 -> xyz=-0.06 0 0.07 rpy=0 0 0
- joint front_marker_tip_joint: origin xyz=0.105 0 0.045 rpy=0 0 0 -> xyz=0.24 0 0.34 rpy=0 0 0

Commit message: fix S10 lidar frame and NV12 camera forwarding

File: deep_robotics/lynx_s10/resource/S10.urdf (robot description, URDF)
Before this commit: robot S10, 24 links, 23 joints
Joints:
- joint front_marker_tip_joint: origin xyz=0.24 0 0.34 rpy=0 0 0 -> xyz=0 0 0.20 rpy=0 0 0; parent base_link -> front_lidar_link
