Commit message: feat(s10-pro): merge Lynx control and media driver

File: deep_robotics/s10_pro/s10_skeleton.urdf (robot description, URDF)
Before this commit: robot deep_robotics_s10_pro_skeleton, 21 links, 20 joints
Links:
- removed link head_direction_left
- removed link head_direction_right
- removed link head_direction_tip
- removed link head_direction_tip_cap
- added link back_lidar_link
- added link front_lidar_link
- added link front_marker_close
- added link front_marker_left
- added link front_marker_right
- added link front_marker_tip
- added link imu_link
- link base_link: mass None -> 8.023087; geometry collision box size=0.16 0.048 0.60; collision cylinder length=0.60 radius=0.08
- link fl_hipx: mass None -> 0.627405; geometry collision cylinder length=0.10 radius=0.04; visual mesh filename=./meshes/fl_hipx.STL
- link fl_hipy: mass None -> 0.885874; geometry collision box size=0.064 0.024 0.18; collision cylinder length=0.080 radius=0.04
- link fl_knee: mass None -> 0.640283; geometry collision box size=0.058 0.020 0.18; collision cylinder length=0.05 radius=0.04
- link fl_wheel: mass None -> 0.587952; geometry collision cylinder length=0.037 radius=0.081; visual mesh filename=./meshes/fl_wheel.STL
- link fr_hipx: mass None -> 0.626546; geometry collision cylinder length=0.10 radius=0.04; visual mesh filename=./meshes/fr_hipx.STL
- link fr_hipy: mass None -> 0.885874; geometry collision box size=0.064 0.024 0.18; collision cylinder length=0.080 radius=0.04
- link fr_knee: mass None -> 0.640283; geometry collision box size=0.058 0.020 0.18; collision cylinder length=0.05 radius=0.04
- link fr_wheel: mass None -> 0.587952; geometry collision cylinder length=0.037 radius=0.081; visual mesh filename=./meshes/fr_wheel.STL
- link hl_hipx: mass None -> 0.626546; geometry collision cylinder length=0.10 radius=0.04; visual mesh filename=./meshes/hl_hipx.STL
- link hl_hipy: mass None -> 0.885874; geometry collision box size=0.064 0.024 0.18; collision cylinder length=0.080 radius=0.04
- link hl_knee: mass None -> 0.640283; geometry collision box size=0.058 0.020 0.18; collision cylinder length=0.05 radius=0.04
- link hl_wheel: mass None -> 0.587952; geometry collision cylinder length=0.037 radius=0.081; visual mesh filename=./meshes/hl_wheel.STL
- link hr_hipx: mass None -> 0.627405; geometry collision cylinder length=0.10 radius=0.04; visual mesh filename=./meshes/hr_hipx.STL
- link hr_hipy: mass None -> 0.885874; geometry collision box size=0.064 0.024 0.18; collision cylinder length=0.080 radius=0.04
- link hr_knee: mass None -> 0.640283; geometry collision box size=0.058 0.020 0.18; collision cylinder length=0.05 radius=0.04
- link hr_wheel: mass None -> 0.587952; geometry collision cylinder length=0.037 radius=0.081; visual mesh filename=./meshes/hr_wheel.STL
Joints:
- removed joint head_direction_left_fixed
- removed joint head_direction_right_fixed
- removed joint head_direction_tip_cap_fixed
- removed joint head_direction_tip_fixed
- added joint back_lidar_joint: type fixed, parent base_link, child back_lidar_link, origin xyz=-0.22341 0.0 -0.0001 rpy=0 0 3.14159
- added joint front_lidar_joint: type fixed, parent base_link, child front_lidar_link, origin xyz=0.22341 0.0 -0.0001 rpy=0 0 0
- added joint front_marker_close_joint: type fixed, parent front_marker_right, child front_marker_close, origin xyz=0.12 0 0 rpy=0 0 0
- added joint front_marker_left_joint: type fixed, parent front_marker_tip, child front_marker_left, origin xyz=-0.06 0 -0.035 rpy=0 0 0
- added joint front_marker_right_joint: type fixed, parent front_marker_left, child front_marker_right, origin xyz=-0.06 0 0.07 rpy=0 0 0
- added joint front_marker_tip_joint: type fixed, parent front_lidar_link, child front_marker_tip, origin xyz=0 0 0.20 rpy=0 0 0
- added joint imu_joint: type fixed, parent base_link, child imu_link, origin xyz=0.0075 -0.0373 0.0556 rpy=1.57 1.57 0
- joint fl_hipx_joint: limit (none) -> lower=-0.6109 upper=0.6109 effort=50.00 velocity=25.76
- joint fl_hipy_joint: limit (none) -> lower=-2.5307 upper=2.5307 effort=50.00 velocity=25.76; origin xyz=0 0.0779 0 rpy=0 0.35 0 -> xyz=0 0.0779 0 rpy=0 0 0
- joint fl_knee_joint: limit (none) -> lower=-2.7227 upper=2.7227 effort=50.00 velocity=25.76; origin xyz=0 0 -0.18 rpy=0 -0.65 0 -> xyz=0 0 -0.18 rpy=0 0 0
- joint fl_wheel_joint: limit (none) -> effort=14.00 velocity=65.50; type revolute -> continuous
- joint fr_hipx_joint: limit (none) -> lower=-0.6109 upper=0.6109 effort=50.00 velocity=25.76
- joint fr_hipy_joint: limit (none) -> lower=-2.5307 upper=2.5307 effort=50.00 velocity=25.76; origin xyz=0 -0.0779 0 rpy=0 0.35 0 -> xyz=0 -0.0779 0 rpy=0 0 0
- joint fr_knee_joint: limit (none) -> lower=-2.7227 upper=2.7227 effort=50.00 velocity=25.76; origin xyz=0 0 -0.18 rpy=0 -0.65 0 -> xyz=0 0 -0.18 rpy=0 0 0
- joint fr_wheel_joint: limit (none) -> effort=14.00 velocity=65.50; type revolute -> continuous
- joint hl_hipx_joint: limit (none) -> lower=-0.6109 upper=0.6109 effort=50.00 velocity=25.76
- joint hl_hipy_joint: limit (none) -> lower=-2.5307 upper=2.5307 effort=50.00 velocity=25.76; origin xyz=0 0.0779 0 rpy=0 -0.35 0 -> xyz=0 0.0779 0 rpy=0 0 0
- joint hl_knee_joint: limit (none) -> lower=-2.7227 upper=2.7227 effort=50.00 velocity=25.76; origin xyz=0 0 -0.18 rpy=0 0.65 0 -> xyz=0 0 -0.18 rpy=0 0 0
- joint hl_wheel_joint: limit (none) -> effort=14.00 velocity=65.50; type revolute -> continuous
- joint hr_hipx_joint: limit (none) -> lower=-0.6109 upper=0.6109 effort=50.00 velocity=25.76
- joint hr_hipy_joint: limit (none) -> lower=-2.5307 upper=2.5307 effort=50.00 velocity=25.76; origin xyz=0 -0.0779 0 rpy=0 -0.35 0 -> xyz=0 -0.0779 0 rpy=0 0 0
- joint hr_knee_joint: limit (none) -> lower=-2.7227 upper=2.7227 effort=50.00 velocity=25.76; origin xyz=0 0 -0.18 rpy=0 0.65 0 -> xyz=0 0 -0.18 rpy=0 0 0
- joint hr_wheel_joint: limit (none) -> effort=14.00 velocity=65.50; type revolute -> continuous
